File: BlinkyHeart.kicad_pcb (KiCad board)
At the start: 2 copper layers, 48.5 x 40.7 mm, 41 parts, among them J1 AVR-ISP-6, SW1 MSK12C02, U1 ATTINY85-20SU, U3 AP3012KTR-G1

Commit message: silkscreen update
Parts:
- moved S1 3.14 mm to (116.8, 82.5)
- moved Logo1 1.09 mm to (119.3, 74.0)
Routing:
- net MISO: track 17.3 -> 19.2 mm
Other:
- board text added: "BlinkyHeart v1.0.0 Tweety's Wild Thinking 2023 github.com/TweetyDaBird"
- board text removed: "Tweety's Wild Thinking - 2023 github.com/TweetyDaBird"
Changed lines of the file:
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@@
   )
   (footprint "TS-1187A:SW_TS-1187A-B-A-B" (layer "F.Cu")
-    (at 117.07 85.68)
+    (at 116.84 82.55)
     (property "LCSC" "C318884")
     (property "MANUFACTURER" "XKB Industrial Precision")
@@
   )
   (footprint "Logotypes:CC_BY_SA_40" (layer "B.Cu")
-    (at 118.630304 74.776725 180)
+    (at 119.340304 73.951725 180)
     (property "Sheetfile" "heart.kicad_sch")
     (property "Sheetname" "")
@@
       (effects (font (size 0.8 0.8) (thickness 0.15)) (justify mirror))
     )
-    (fp_text value "CC-BY-SA-4.0" (at -14.469696 1.386725) (layer "B.SilkS")
+    (fp_text value "CC-BY-SA-4.0" (at 0 -1.43) (layer "B.SilkS")
       (effects (font (size 0.8 0.8) (thickness 0.15)) (justify mirror))
     )
-    (fp_text user "https://creativecommons.org" (at -14.469696 0.276725) (layer "B.SilkS")
+    (fp_text user "https://creativecommons.org" (at 0 -2.54) (layer "B.SilkS") hide
       (effects (font (size 0.8 0.8) (thickness 0.15)) (justify mirror))
     )
@@
     (effects (font (size 1 1) (thickness 0.15)) (justify mirror))
   )
-  (gr_text "Tweety's Wild Thinking - 2023\ngithub.com/TweetyDaBird\n" (at 119.82 79.9) (layer "F.SilkS")
-    (effects (font (size 1 1) (thickness 0.15)))
+  (gr_text "BlinkyHeart v1.0.0\nTweety's Wild Thinking 2023\ngithub.com/TweetyDaBird\n" (at 137.16 73.66) (layer "B.SilkS")
+    (effects (font (size 1 1) (thickness 0.15)) (justify mirror))
   )
-  (segment (start 120.07 83.805) (end 122.35 83.805) (width 0.25) (layer "F.Cu") (net 2))
-  (segment (start 122.35 83.805) (end 124.845 86.3) (width 0.25) (layer "F.Cu") (net 2))
+  (segment (start 119.84 81.295) (end 124.845 86.3) (width 0.25) (layer "F.Cu") (net 2))
   (segment (start 122.575 89.915) (end 123.225 90.565) (width 0.25) (layer "F.Cu") (net 2))
-  (segment (start 114.07 83.805) (end 120.07 83.805) (width 0.25) (layer "F.Cu") (net 2))
   (segment (start 122.575 88.575) (end 122.575 89.915) (width 0.25) (layer "F.Cu") (net 2))
   (segment (start 124.85 86.3) (end 122.575 88.575) (width 0.25) (layer "F.Cu") (net 2))
+  (segment (start 113.84 80.675) (end 119.84 80.675) (width 0.25) (layer "F.Cu") (net 2))
+  (segment (start 119.84 80.675) (end 119.84 81.295) (width 0.25) (layer "F.Cu") (net 2))
   (segment (start 143.524143 71.040834) (end 143.524143 72.424143) (width 0.45) (layer "F.Cu") (net 3))
   (segment (start 131.317059 99.972941) (end 131.012758 99.972941) (width 0.45) (layer "F.Cu") (net 3))
